File: controller/penguin.kicad_pcb (KiCad board)
At the start: 4 copper layers, 89.5 x 62.6 mm, 165 parts, among them IC1 HY2120-AB, J1 USB_C_CONN, J10 MTR_HEADER_2, J2 CAM_HEADER, J3 BATT_BALANCE_HEADER, J4 TOF_HEADER, J5 I2C_JUMPER, J6 I2C_JUMPER, J7 SERVO_CONN, J8 BATT_CONN, J9 MTR_HEADER_1, Q1 AO3400A, Q2 SI2393DS, Q3 2N7002, Q4 FS8205A, SW1 SW_Boot, SW2 SW_Reset, U1 ESP32-S3-WROOM-1U-N8R8, U10 TPS62143, U2 LP5907MFX-2.8, U3 LP5907MFX-1.2, U4 DRV8833PW, U5 MCP23017_ML, U6 TPS5405DR, U7 AMS1117-3.3, U8 DMP4065S-7, U9 LSM6DSL

Commit message: cam testing
Routing:
- net Net-(J2-Pin_1): vias 0 -> 2
- net GND: vias 362 -> 358
- net CAM_D9: vias 0 -> 2
Changed lines of the file:
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@@
 		(tags "connector Hirose FH12 horizontal")
 		(property "Reference" "J2"
-			(at 0 0.95 180)
+			(at 0 0.95 360)
 			(layer "F.SilkS")
 			(effects
@@
 		)
 		(property "Value" "CAM_HEADER"
-			(at 0 5.6 0)
+			(at 0 5.6 360)
 			(layer "F.Fab")
 			(effects
@@
 		)
 		(fp_text user "${REFERENCE}"
-			(at 0 3.7 0)
+			(at 0 3.7 360)
 			(layer "F.Fab")
 			(effects
@@
 	)
 	(via
-		(at 136.925 114.95)
-		(size 0.6)
-		(drill 0.3)
-		(layers "F.Cu" "B.Cu")
-		(net 2)
-	)
-	(via
 		(at 180.8 64.325)
 		(size 0.6)
@@
 	)
 	(via
-		(at 137.675 114.95)
-		(size 0.6)
-		(drill 0.3)
-		(layers "F.Cu" "B.Cu")
-		(net 2)
-	)
-	(via
 		(at 179.475 108.1)
 		(size 0.6)
@@
 	)
 	(via
-		(at 146.73 115.8)
-		(size 0.6)
-		(drill 0.3)
-		(layers "F.Cu" "B.Cu")
-		(net 2)
-	)
-	(via
 		(at 115.4625 98.34)
 		(size 0.6)
@@
 	)
 	(via
-		(at 147.48 115.8)
-		(size 0.6)
-		(drill 0.3)
-		(layers "F.Cu" "B.Cu")
-		(net 2)
-	)
-	(via
 		(at 108.85 99.75)
 		(size 0.6)
@@
 		(net 48)
 	)
+	(via
+		(at 146.73 115.8)
+		(size 0.6)
+		(drill 0.3)
+		(layers "F.Cu" "B.Cu")
+		(net 48)
+	)
+	(via
+		(at 147.48 115.8)
+		(size 0.6)
+		(drill 0.3)
+		(layers "F.Cu" "B.Cu")
+		(net 48)
+	)
 	(segment
 		(start 143.41 105.7525)
@@
 		(net 128)
 	)
+	(via
+		(at 136.925 114.95)
+		(size 0.6)
+		(drill 0.3)
+		(layers "F.Cu" "B.Cu")
+		(net 128)
+	)
+	(via
+		(at 137.675 114.95)
+		(size 0.6)
+		(drill 0.3)
+		(layers "F.Cu" "B.Cu")
+		(net 128)
+	)

Commit message: bug fixes, change servo constants from degrees to us
Routing:
- net Net-(J2-Pin_1): vias 2 -> 0
- net GND: vias 358 -> 362
- net CAM_D9: vias 2 -> 0
Changed lines of the file:
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@@
 			(layer "F.Mask"
 				(type "Top Solder Mask")
+				(color "#000101D4")
 				(thickness 0.01)
 			)
@@
 			(layer "B.Mask"
 				(type "Bottom Solder Mask")
+				(color "#000101D4")
 				(thickness 0.01)
 			)
@@
 				(type "Bottom Silk Screen")
 			)
-			(copper_finish "None")
+			(copper_finish "HAL SnPb")
 			(dielectric_constraints no)
 		)
@@
 		(tags "connector Hirose FH12 horizontal")
 		(property "Reference" "J2"
-			(at 0 0.95 360)
+			(at 0 0.95 0)
 			(layer "F.SilkS")
 			(effects
@@
 		)
 		(property "Value" "CAM_HEADER"
-			(at 0 5.6 360)
+			(at 0 5.6 0)
 			(layer "F.Fab")
 			(effects
@@
 		)
 		(fp_text user "${REFERENCE}"
-			(at 0 3.7 360)
+			(at 0 3.7 0)
 			(layer "F.Fab")
 			(effects
@@
 	)
 	(via
+		(at 136.925 114.95)
+		(size 0.6)
+		(drill 0.3)
+		(layers "F.Cu" "B.Cu")
+		(net 2)
+	)
+	(via
 		(at 180.8 64.325)
 		(size 0.6)
@@
 	)
 	(via
+		(at 137.675 114.95)
+		(size 0.6)
+		(drill 0.3)
+		(layers "F.Cu" "B.Cu")
+		(net 2)
+	)
+	(via
 		(at 179.475 108.1)
 		(size 0.6)
@@
 	)
 	(via
+		(at 146.73 115.8)
+		(size 0.6)
+		(drill 0.3)
+		(layers "F.Cu" "B.Cu")
+		(net 2)
+	)
+	(via
 		(at 115.4625 98.34)
 		(size 0.6)
@@
 	)
 	(via
+		(at 147.48 115.8)
+		(size 0.6)
+		(drill 0.3)
+		(layers "F.Cu" "B.Cu")
+		(net 2)
+	)
+	(via
 		(at 108.85 99.75)
 		(size 0.6)
@@
 		(net 48)
 	)
-	(via
-		(at 146.73 115.8)
-		(size 0.6)
-		(drill 0.3)
-		(layers "F.Cu" "B.Cu")
-		(net 48)
-	)
-	(via
-		(at 147.48 115.8)
-		(size 0.6)
-		(drill 0.3)
-		(layers "F.Cu" "B.Cu")
-		(net 48)
-	)
 	(segment
 		(start 143.41 105.7525)
@@
 		(net 128)
 	)
-	(via
-		(at 136.925 114.95)
-		(size 0.6)
-		(drill 0.3)
-		(layers "F.Cu" "B.Cu")
-		(net 128)
-	)
-	(via
-		(at 137.675 114.95)
-		(size 0.6)
-		(drill 0.3)
-		(layers "F.Cu" "B.Cu")
-		(net 128)
-	)
